File: learning/led_matrix_array/led_matrix_array.kicad_pcb (KiCad board)
At the start: 2 copper layers, 113.8 x 61.5 mm, 21 parts, among them J1 Barrel_Jack, J2 LED1_IN, J3 LED1_OUT, J4 LED2_IN, J5 LED2_OUT, J6 LED3_IN, J7 LED3_OUT, J8 LED4_IN, J9 LED4_OUT, U1 ArduinoProMiniSimple

Commit message: Setup of schematic editor for a new project
Connections:
- J2 pad 1: /CS0 -> /CLK0
- J2 pad 2: /DIN0 -> /CS0
- J2 pad 3: /CLK0 -> /DIN0
- J3 pad 1: /CS1 -> /CLK1
- J3 pad 2: /DIN1 -> /CS1
- J3 pad 3: /CLK1 -> /DIN1
- J4 pad 1: /CS1 -> /CLK1
- J4 pad 2: /DIN1 -> /CS1
- J4 pad 3: /CLK1 -> /DIN1
- J5 pad 1: /CS2 -> /CLK2
- J5 pad 2: /DIN2 -> /CS2
- J5 pad 3: /CLK2 -> /DIN2
- J6 pad 1: /CS2 -> /CLK2
- J6 pad 2: /DIN2 -> /CS2
- J6 pad 3: /CLK2 -> /DIN2
- J7 pad 1: /CS3 -> /CLK3
- J7 pad 2: /DIN3 -> /CS3
- J7 pad 3: /CLK3 -> /DIN3
- J8 pad 1: /CS3 -> /CLK3
- J8 pad 2: /DIN3 -> /CS3
- J8 pad 3: /CLK3 -> /DIN3
- U1 pad 15: /DIN0 -> /CS0
- U1 pad 16: /CLK0 -> /DIN0
- U1 pad 18: /CS0 -> /CLK0
Routing:
- net /CS0: track 37.5 -> 32.1 mm, vias 2 -> 0
- net /DIN0: track 32.1 -> 37.1 mm
- net /CS1: track 72.0 -> 70.3 mm
- net /CLK2: track 75.8 -> 74.8 mm
- net /CLK1: track 71.0 -> 72.0 mm
- net /DIN1: track 70.3 -> 71.0 mm
- net /CS2: track 74.8 -> 75.4 mm
- net /CLK0: track 37.1 -> 37.5 mm, vias 0 -> 2
