File: learning/led_matrix_array/led_matrix_array.kicad_sch (KiCad schematic)
At the start: 19 parts, among them J1 Barrel_Jack, J2 LED1_IN, J3 LED1_OUT, J4 LED2_IN, J5 LED2_OUT, J6 LED3_IN, J7 LED3_OUT, J8 LED4_IN, J9 LED4_OUT, U1 ArduinoProMiniSimple

Commit message: Setup of schematic editor for a new project
Connections:
- net CLK0: now also J2.1 (Pin_1), U1.18 (13); no longer J2.3 (Pin_3), U1.16 (11)
- net CLK1: now also J3.1 (Pin_1), J4.1 (Pin_1); no longer J3.3 (Pin_3), J4.3 (Pin_3)
- net CLK2: now also J5.1 (Pin_1), J6.1 (Pin_1); no longer J5.3 (Pin_3), J6.3 (Pin_3)
- net CLK3: now also J7.1 (Pin_1), J8.1 (Pin_1); no longer J7.3 (Pin_3), J8.3 (Pin_3)
- net CS0: now also J2.2 (Pin_2), U1.15 (10); no longer J2.1 (Pin_1), U1.18 (13)
- net CS1: now also J3.2 (Pin_2), J4.2 (Pin_2); no longer J3.1 (Pin_1), J4.1 (Pin_1)
- net CS2: now also J5.2 (Pin_2), J6.2 (Pin_2); no longer J5.1 (Pin_1), J6.1 (Pin_1)
- net CS3: now also J7.2 (Pin_2), J8.2 (Pin_2); no longer J7.1 (Pin_1), J8.1 (Pin_1)
- net DIN0: now also J2.3 (Pin_3), U1.16 (11); no longer J2.2 (Pin_2), U1.15 (10)
- net DIN1: now also J3.3 (Pin_3), J4.3 (Pin_3); no longer J3.2 (Pin_2), J4.2 (Pin_2)
- net DIN2: now also J5.3 (Pin_3), J6.3 (Pin_3); no longer J5.2 (Pin_2), J6.2 (Pin_2)
- net DIN3: now also J7.3 (Pin_3), J8.3 (Pin_3); no longer J7.2 (Pin_2), J8.2 (Pin_2)
Changed lines of the file:
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@@
 	)
 	(label "DIN1"
-		(at 168.91 100.33 0)
+		(at 168.91 97.79 0)
 		(effects
 			(font
@@
 	)
 	(label "DIN0"
-		(at 132.08 100.33 0)
+		(at 132.08 97.79 0)
 		(effects
 			(font
@@
 	)
 	(label "CLK0"
-		(at 132.08 97.79 0)
+		(at 132.08 105.41 0)
 		(effects
 			(font
@@
 	)
 	(label "CS0"
-		(at 132.08 105.41 0)
+		(at 132.08 100.33 0)
 		(effects
 			(font
@@
 	)
 	(label "CLK1"
-		(at 168.91 97.79 0)
+		(at 168.91 102.87 0)
 		(effects
 			(font
@@
 	)
 	(label "CLK3"
+		(at 227.33 102.87 0)
+		(effects
+			(font
+				(size 1.27 1.27)
+			)
+			(justify left bottom)
+		)
+	)
+	(label "CS2"
+		(at 198.12 100.33 0)
+		(effects
+			(font
+				(size 1.27 1.27)
+			)
+			(justify left bottom)
+		)
+	)
+	(label "GND"
+		(at 86.36 62.23 0)
+		(effects
+			(font
+				(size 1.27 1.27)
+			)
+			(justify left bottom)
+		)
+	)
+	(label "Vcc"
+		(at 168.91 92.71 0)
+		(effects
+			(font
+				(size 1.27 1.27)
+			)
+			(justify left bottom)
+		)
+	)
+	(label "DIN2"
+		(at 198.12 97.79 0)
+		(effects
+			(font
+				(size 1.27 1.27)
+			)
+			(justify left bottom)
+		)
+	)
+	(label "Vcc"
+		(at 146.05 92.71 180)
+		(effects
+			(font
+				(size 1.27 1.27)
+			)
+			(justify right bottom)
+		)
+	)
+	(label "CS1"
+		(at 168.91 100.33 0)
+		(effects
+			(font
+				(size 1.27 1.27)
+			)
+			(justify left bottom)
+		)
+	)
+	(label "Vcc"
+		(at 198.12 92.71 0)
+		(effects
+			(font
+				(size 1.27 1.27)
+			)
+			(justify left bottom)
+		)
+	)
+	(label "GND"
+		(at 227.33 95.25 0)
+		(effects
+			(font
+				(size 1.27 1.27)
+			)
+			(justify left bottom)
+		)
+	)
+	(label "GND"
+		(at 86.36 116.84 270)
+		(effects
+			(font
+				(size 1.27 1.27)
+			)
+			(justify right bottom)
+		)
+	)
+	(label "Vcc"
+		(at 93.98 148.59 0)
+		(effects
+			(font
+				(size 1.27 1.27)
+			)
+			(justify left bottom)
+		)
+	)
+	(label "CS3"
+		(at 227.33 100.33 0)
+		(effects
+			(font
+				(size 1.27 1.27)
+			)
+			(justify left bottom)
+		)
+	)
+	(label "CLK2"
+		(at 198.12 102.87 0)
+		(effects
+			(font
+				(size 1.27 1.27)
+			)
+			(justify left bottom)
+		)
+	)
+	(label "DIN3"
 		(at 227.33 97.79 0)
 		(effects
 			(font
-				(size 1.27 1.27)
-			)
-			(justify left bottom)
-		)
-	)
-	(label "CS2"
-		(at 198.12 102.87 0)
-		(effects
-			(font
-				(size 1.27 1.27)
-			)
-			(justify left bottom)
-		)
-	)
-	(label "GND"
-		(at 86.36 62.23 0)
-		(effects
-			(font
-				(size 1.27 1.27)
-			)
-			(justify left bottom)
-		)
-	)
-	(label "Vcc"
-		(at 168.91 92.71 0)
-		(effects
-			(font
-				(size 1.27 1.27)
-			)
-			(justify left bottom)
-		)
-	)
-	(label "DIN2"
-		(at 198.12 100.33 0)
-		(effects
-			(font
-				(size 1.27 1.27)
-			)
-			(justify left bottom)
-		)
-	)
-	(label "Vcc"
-		(at 146.05 92.71 180)
-		(effects
-			(font
-				(size 1.27 1.27)
-			)
-			(justify right bottom)
-		)
-	)
-	(label "CS1"
-		(at 168.91 102.87 0)
-		(effects
-			(font
-				(size 1.27 1.27)
-			)
-			(justify left bottom)
-		)
-	)
-	(label "Vcc"
-		(at 198.12 92.71 0)
-		(effects
-			(font
-				(size 1.27 1.27)
-			)
-			(justify left bottom)
-		)
-	)
-	(label "GND"
-		(at 227.33 95.25 0)
-		(effects
-			(font
-				(size 1.27 1.27)
-			)
-			(justify left bottom)
-		)
-	)
-	(label "GND"
-		(at 86.36 116.84 270)
-		(effects
-			(font
-				(size 1.27 1.27)
-			)
-			(justify right bottom)
-		)
-	)
-	(label "Vcc"
-		(at 93.98 148.59 0)
-		(effects
-			(font
-				(size 1.27 1.27)
-			)
-			(justify left bottom)
-		)
-	)
-	(label "CS3"
-		(at 227.33 102.87 0)
-		(effects
-			(font
-				(size 1.27 1.27)
-			)
-			(justify left bottom)
-		)
-	)
-	(label "CLK2"
-		(at 198.12 97.79 0)
-		(effects
-			(font
-				(size 1.27 1.27)
-			)
-			(justify left bottom)
-		)
-	)
-	(label "DIN3"
-		(at 227.33 100.33 0)
-		(effects
-			(font
